File: DarkQuest_A5202_Adapter.kicad_sch (KiCad schematic)
At the start: 18 parts, among them J1 HSEC8-170-01-X-DV-A, J10 RJ45_Shielded, J11 RJ45_Shielded, J12 RJ45_Shielded, J13 RJ45_Shielded, J14 RJ45_Shielded, J15 RJ45_Shielded, J16 RJ45_Shielded, J17 RJ45_Shielded, J18 Conn_01x02_Pin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

Commit message: RJ45v1
Connections:
- net A32: now also J10.8; no longer J10.2
- net A33: now also J11.2; no longer J10.6
- net A34: now also J10.6; no longer J10.4
- net A35: now also J11.4; no longer J10.8
- net A36: now also J10.4; no longer J11.2
- net A38: now also J10.2; no longer J11.4
- net A40: now also J12.8; no longer J12.2
- net A41: now also J13.2; no longer J12.6
- net A42: now also J12.6; no longer J12.4
- net A43: now also J13.4; no longer J12.8
- net A44: now also J12.4; no longer J13.2
- net A46: now also J12.2; no longer J13.4
- net A48: now also J14.8; no longer J14.2
- net A49: now also J15.2; no longer J14.6
- net A50: now also J14.6; no longer J14.4
- net A51: now also J15.4; no longer J14.8
- net A52: now also J14.4; no longer J15.2
- net A54: now also J14.2; no longer J15.4
- net A56: now also J16.8; no longer J16.2
- net A57: now also J17.2; no longer J16.6
- net A58: now also J16.6; no longer J16.4
- net A59: now also J17.4; no longer J16.8
- net A60: now also J16.4; no longer J17.2
- net A62: now also J16.2; no longer J17.4
- net K32: now also J10.7; no longer J10.1
- net K33: now also J11.1; no longer J10.3
- net K34: now also J10.3; no longer J10.5
- net K35: now also J11.5; no longer J10.7
- net K36: now also J10.5; no longer J11.1
- net K38: now also J10.1; no longer J11.5
- net K40: now also J12.7; no longer J12.1
- net K41: now also J13.1; no longer J12.3
- net K42: now also J12.3; no longer J12.5
- net K43: now also J13.5; no longer J12.7
- net K44: now also J12.5; no longer J13.1
- net K46: now also J12.1; no longer J13.5
- net K48: now also J14.7; no longer J14.1
- net K49: now also J15.1; no longer J14.3
- net K50: now also J14.3; no longer J14.5
- net K51: now also J15.5; no longer J14.7
- net K52: now also J14.5; no longer J15.1
- net K54: now also J14.1; no longer J15.5
- net K56: now also J16.7; no longer J16.1
- net K57: now also J17.1; no longer J16.3
- net K58: now also J16.3; no longer J16.5
- net K59: now also J17.5; no longer J16.7
- net K60: now also J16.5; no longer J17.1
- net K62: now also J16.1; no longer J17.5
Changed lines of the file:
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@@
 		)
 	)
-	(label "A50"
+	(label "A52"
 		(at 184.15 140.97 180)
 		(effects
@@
 		)
 	)
-	(label "A40"
+	(label "A46"
 		(at 234.95 111.76 180)
 		(effects
@@
 		)
 	)
-	(label "K35"
+	(label "K32"
 		(at 184.15 99.06 180)
 		(effects
@@
 		)
 	)
-	(label "K62"
+	(label "K59"
 		(at 273.05 138.43 0)
 		(effects
@@
 		)
 	)
-	(label "K38"
+	(label "K35"
 		(at 222.25 104.14 0)
 		(effects
@@
 		)
 	)
-	(label "A49"
+	(label "A50"
 		(at 184.15 135.89 180)
 		(effects
@@
 		)
 	)
-	(label "K58"
+	(label "K60"
 		(at 234.95 138.43 180)
 		(effects
@@
 		)
 	)
-	(label "A58"
+	(label "A60"
 		(at 234.95 140.97 180)
 		(effects
@@
 		)
 	)
-	(label "A41"
+	(label "A42"
 		(at 234.95 101.6 180)
 		(effects
@@
 		)
 	)
-	(label "K57"
+	(label "K58"
 		(at 234.95 143.51 180)
 		(effects
@@
 		)
 	)
-	(label "K32"
+	(label "K38"
 		(at 184.15 114.3 180)
 		(effects
@@
 		)
 	)
-	(label "A35"
+	(label "A32"
 		(at 184.15 96.52 180)
 		(effects
@@
 		)
 	)
-	(label "A46"
+	(label "A43"
 		(at 273.05 106.68 0)
 		(effects
@@
 		)
 	)
-	(label "K43"
+	(label "K40"
 		(at 234.95 99.06 180)
 		(effects
@@
 		)
 	)
-	(label "K34"
+	(label "K36"
 		(at 184.15 104.14 180)
 		(effects
@@
 		)
 	)
-	(label "A62"
+	(label "A59"
 		(at 273.05 140.97 0)
 		(effects
@@
 		)
 	)
-	(label "K33"
+	(label "K34"
 		(at 184.15 109.22 180)
 		(effects
@@
 		)
 	)
-	(label "K49"
+	(label "K50"
 		(at 184.15 143.51 180)
 		(effects
@@
 		)
 	)
-	(label "A33"
+	(label "A34"
 		(at 184.15 101.6 180)
 		(effects
@@
 		)
 	)
-	(label "A44"
+	(label "A41"
 		(at 273.05 111.76 0)
 		(effects
@@
 		)
 	)
-	(label "K36"
+	(label "K33"
 		(at 222.25 114.3 0)
 		(effects
@@
 		)
 	)
-	(label "A34"
+	(label "A36"
 		(at 184.15 106.68 180)
 		(effects
@@
 		)
 	)
-	(label "K42"
+	(label "K44"
 		(at 234.95 104.14 180)
 		(effects
@@
 		)
 	)
-	(label "A59"
+	(label "A56"
 		(at 234.95 130.81 180)
 		(effects
@@
 		)
 	)
-	(label "K54"
+	(label "K51"
 		(at 222.25 138.43 0)
 		(effects
@@
 		)
 	)
-	(label "A48"
+	(label "A54"
 		(at 184.15 146.05 180)
 		(effects
@@
 		)
 	)
-	(label "K59"
+	(label "K56"
 		(at 234.95 133.35 180)
 		(effects
@@
 		)
 	)
-	(label "A60"
+	(label "A57"
 		(at 273.05 146.05 0)
 		(effects
@@
 		)
 	)
+	(label "K42"
+		(at 234.95 109.22 180)
+		(effects
+			(font
+				(size 1.27 1.27)
+			)
+			(justify right bottom)
+		)
+	)
 	(label "K41"
-		(at 234.95 109.22 180)
-		(effects
-			(font
-				(size 1.27 1.27)
-			)
-			(justify right bottom)
-		)
-	)
-	(label "K44"
 		(at 273.05 114.3 0)
 		(effects
@@
 		)
 	)
-	(label "K40"
+	(label "K46"
 		(at 234.95 114.3 180)
 		(effects
@@
 		)
 	)
-	(label "A51"
+	(label "A48"
 		(at 184.15 130.81 180)
 		(effects
@@
 		)
 	)
-	(label "K50"
+	(label "K52"
 		(at 184.15 138.43 180)
 		(effects
@@
 		)
 	)
-	(label "A38"
+	(label "A35"
 		(at 222.25 106.68 0)
 		(effects
@@
 		)
 	)
-	(label "K48"
+	(label "K54"
 		(at 184.15 148.59 180)
 		(effects
@@
 		)
 	)
-	(label "K51"
+	(label "K48"
 		(at 184.15 133.35 180)
 		(effects
@@
 		)
 	)
-	(label "A54"
+	(label "A51"
 		(at 222.25 140.97 0)
 		(effects
@@
 		)
 	)
-	(label "A36"
+	(label "A33"
 		(at 222.25 111.76 0)
 		(effects
@@
 		)
 	)
-	(label "K60"
+	(label "K57"
 		(at 273.05 148.59 0)
 		(effects
@@
 		)
 	)
-	(label "A57"
+	(label "A58"
 		(at 234.95 135.89 180)
 		(effects
@@
 		)
 	)
-	(label "A42"
+	(label "A44"
 		(at 234.95 106.68 180)
 		(effects
@@
 		)
 	)
-	(label "A32"
+	(label "A38"
 		(at 184.15 111.76 180)
 		(effects
@@
 		)
 	)
-	(label "A43"
+	(label "A40"
 		(at 234.95 96.52 180)
 		(effects
@@
 		)
 	)
-	(label "K56"
+	(label "K62"
 		(at 234.95 148.59 180)
 		(effects
@@
 		)
 	)
-	(label "A52"
+	(label "A49"
 		(at 222.25 146.05 0)
 		(effects
@@
 		)
 	)
-	(label "A56"
+	(label "A62"
 		(at 234.95 146.05 180)
 		(effects
@@
 		)
 	)
-	(label "K46"
+	(label "K43"
 		(at 273.05 104.14 0)
 		(effects
@@
 		)
 	)
-	(label "K52"
+	(label "K49"
 		(at 222.25 148.59 0)
 		(effects
